Commit message: add robot_model
model

File: my_robot_model/urdf/my_robo_hardware.xacro (robot description, xacro)
@@ -106,5 +106,5 @@
   <!--========================================== LEFT WHEEL JOINT ==========================================-->
   <joint name="left_wheel_joint" type="continuous">
-    <origin xyz="0.0 -0.158075 0.065" rpy="0.0 0.0 0.0"/>
+    <origin xyz="0.0 0.158075 0.065" rpy="0.0 0.0 0.0"/>
     <parent link="base_link" />
     <child link="left_wheel_link" />
@@ -146,5 +146,5 @@
 <!--========================================== RIGHT WHEEL JOINT ==========================================-->
 <joint name="right_wheel_joint" type="continuous">
-  <origin xyz="0.0 0.158075 0.065" rpy="0 0.0 0.0"/>
+  <origin xyz="0.0 -0.158075 0.065" rpy="0 0.0 0.0"/>
   <parent link="base_link" />
   <child link="right_wheel_link" />
@@ -201,5 +201,5 @@
   <!--============================================ FRONT CASTOR WHEEL JOINT ============================================-->
   <joint name="front_castor_wheel_joint" type="fixed">
-    <origin xyz="0.2 0.0 0.0252" rpy="0.0 0.0 0.0"/>
+    <origin xyz="0.2 0.0 0.026" rpy="0.0 0.0 0.0"/>
     <parent link="base_link" />
     <child link="front_castor_wheel_link" />
@@ -245,5 +245,5 @@
   <!--============================================ REAR CASTOR WHEEL JOINT ============================================-->
   <joint name="rear_castor_wheel_joint" type="fixed">
-    <origin xyz="-0.2 0.0 0.0252" rpy="0.0 0.0 0.0"/>
+    <origin xyz="-0.2 0.0 0.026" rpy="0.0 0.0 0.0"/>
     <parent link="base_link" />
     <child link="rear_castor_wheel_link" />

File: my_robot_model/urdf/my_robo_simulation.xacro (robot description, xacro)
@@ -80,5 +80,5 @@
     <parent link="base_footprint" />
     <child link="base_link" />
-    <axis xyz="0 0 0" />
+    <axis xyz="0 1 0" />
   </joint>
   <!--========================================== LEFT WHEEL LINK ==========================================-->
@@ -106,5 +106,5 @@
   <!--========================================== LEFT WHEEL JOINT ==========================================-->
   <joint name="left_wheel_joint" type="continuous">
-    <origin xyz="0.0 -0.158075 0.065" rpy="0.0 0.0 0.0"/>
+    <origin xyz="0.0 0.158075 0.065" rpy="0.0 0.0 0.0"/>
     <parent link="base_link" />
     <child link="left_wheel_link" />
@@ -142,9 +142,24 @@
       <mesh filename="package://robot/urdf/meshes/wheelR.stl" scale="0.1 0.1 0.1"/>
     </geometry>
+    <!-- <surface>
+      <friction>
+        <ode>
+          <mu>0.8</mu>
+          <mu2>0.8</mu2>
+          <slip1>0.0</slip1>
+          <slip2>0.0</slip2>
+        </ode>
+      </friction>
+    </surface> -->
   </collision>
 </link>
+<!-- <gazebo reference="right_wheel_link">
+  <mu1 value="0.8"/>
+  <mu2 value="0.8"/>
+  <slip value="0.0"/>
+</gazebo> -->
 <!--========================================== RIGHT WHEEL JOINT ==========================================-->
 <joint name="right_wheel_joint" type="continuous">
-  <origin xyz="0.0 0.158075 0.065" rpy="0 0.0 0.0"/>
+  <origin xyz="0.0 -0.158075 0.065" rpy="0 0.0 0.0"/>
   <parent link="base_link" />
   <child link="right_wheel_link" />
@@ -201,5 +216,5 @@
   <!--============================================ FRONT CASTOR WHEEL JOINT ============================================-->
   <joint name="front_castor_wheel_joint" type="fixed">
-    <origin xyz="0.2 0.0 0.0252" rpy="0.0 0.0 0.0"/>
+    <origin xyz="0.2 0.0 0.027" rpy="0.0 0.0 0.0"/>
     <parent link="base_link" />
     <child link="front_castor_wheel_link" />
@@ -245,5 +260,5 @@
   <!--============================================ REAR CASTOR WHEEL JOINT ============================================-->
   <joint name="rear_castor_wheel_joint" type="fixed">
-    <origin xyz="-0.2 0.0 0.0252" rpy="0.0 0.0 0.0"/>
+    <origin xyz="-0.2 0.0 0.027" rpy="0.0 0.0 0.0"/>
     <parent link="base_link" />
     <child link="rear_castor_wheel_link" />
@@ -279,26 +294,105 @@
     <axis xyz="0 0 0" />
   </joint>
+  <!--========================================== LIDAR PLUGIN - GAZEBO ==========================================-->
+  <!--Sample size of 4000 (original value of RPLidarA1M8) gives an error-->
+  <gazebo reference="laser_link">
+    <!--sensor type="gpu_ray" name="laser"-->
+    <sensor type="ray" name="laser">
+        <pose>0 0 0 0 0 0</pose>
+        <visualize>false</visualize>
+        <update_rate>40</update_rate>
+        <ray>
+            <scan>
+                <horizontal>
+                    <samples>720</samples>
+                    <resolution>1</resolution>
+                    <min_angle>0</min_angle>
+                    <max_angle>6.28</max_angle>
+                </horizontal>
+            </scan>
+            <range>
+                <min>0.1</min>
+                <max>6</max>
+                <resolution>0.1</resolution>
+            </range>
+        </ray>
+        <!--plugin name="gpu_laser" filename="libgazebo_ros_gpu_laser.so"-->
+        <plugin name="gpu_laser" filename="libgazebo_ros_laser.so">
+            <topicName>/scan</topicName>
+            <frameName>laser_link</frameName>
+        </plugin>
+    </sensor>
+</gazebo>
+      <!--========================================== IMU LINK ==========================================-->
+      <link name="imu_link">
+        <inertial>
+          <origin xyz="0 0 0" rpy="0 0 0" />
+          <mass value="0.0093378" />
+          <inertia ixx="0" ixy="0" ixz="0" iyy="0" iyz="0" izz="0" />
+        </inertial>
+        <visual>
+          <origin xyz="0 0 0" rpy="0 0 0" />
+          <geometry>
+            <box size="0.05 0.01 0.02"/>
+          </geometry>
+          <material name="Red" />
+        </visual>
+        <collision>
+          <origin xyz="0 0 0" rpy="0 0 0" />
+          <geometry>
+            <box size="0.05 0.01 0.02"/>
+          </geometry>
+        </collision>
+      </link>
+      <!--========================================== IMU JOINT ==========================================-->
+      <joint name="imu_joint" type="fixed">
+        <origin xyz="0.0075 0.0 0.25" rpy="0 0 3.14" />
+        <parent link="base_link" />
+        <child link="imu_link" />
+        <axis xyz="0 0 0" />
+      </joint>
+  <!--============================================= IMU PLUGIN - GAZEBO =============================================-->
+  <gazebo reference="imu_link">
+    <gravity>true</gravity>
+    <sensor name="imu_sensor" type="imu">
+      <always_on>true</always_on>
+      <update_rate>100</update_rate>
+      <visualize>true</visualize>
+      <topic>__default_topic__</topic>
+      <plugin filename="libgazebo_ros_imu_sensor.so" name="imu_plugin">
+        <topicName>imu_data</topicName>
+        <bodyName>imu_link</bodyName>
+        <updateRateHZ>10.0</updateRateHZ>
+        <gaussianNoise>0.0</gaussianNoise>
+        <xyzOffset>0 0 0</xyzOffset>
+        <rpyOffset>0 0 0</rpyOffset>
+        <frameName>imu_link</frameName>
+        <initialOrientationAsReference>false</initialOrientationAsReference>
+      </plugin>
+      <pose>0 0 0 0 0 0</pose>
+    </sensor>
+  </gazebo>
   <!--========================================== GAZEBO TAGS ==========================================-->
-  <gazebo reference="base_link">
+  <!-- <gazebo reference="base_link">
     <material>Gazebo/Blue</material>
-  </gazebo>
-  <gazebo reference="robot_body_link">
+  </gazebo> -->
+  <!-- <gazebo reference="robot_body_link">
     <material>Gazebo/Orange</material>
-  </gazebo>
-  <gazebo reference="right_wheel_link">
+  </gazebo> -->
+  <!-- <gazebo reference="right_wheel_link">
     <material>Gazebo/Red</material>
-  </gazebo>
-  <gazebo reference="left_wheel_link">
+  </gazebo> -->
+  <!-- <gazebo reference="left_wheel_link">
     <material>Gazebo/Red</material>
-  </gazebo>
-  <gazebo reference="front_castor_wheel_link">
+  </gazebo> -->
+  <!-- <gazebo reference="front_castor_wheel_link">
     <material>Gazebo/Red</material>
-  </gazebo>
-  <gazebo reference="rear_castor_wheel_link">
+  </gazebo> -->
+  <!-- <gazebo reference="rear_castor_wheel_link">
     <material>Gazebo/Red</material>
-  </gazebo>
-  <gazebo reference="laser_link">
+  </gazebo> -->
+  <!-- <gazebo reference="laser_link">
     <material>Gazebo/Green</material>
-  </gazebo>
+  </gazebo> -->
   <!--========================================== DIFF DRIVE PLUGIN - GAZEBO ==========================================-->
 	<gazebo>
@@ -315,7 +409,7 @@
 		<wheelDiameter>0.13</wheelDiameter>
 		<!-- Wheel acceleration, in rad/s^2, defaults to 0.0 rad/s^2 -->
-		<wheelAcceleration>2</wheelAcceleration>
+		<wheelAcceleration>0.8</wheelAcceleration>
 		<!-- Maximum torque which the wheels can produce, in Nm, defaults to 5 Nm -->
-		<wheelTorque>6</wheelTorque>
+		<wheelTorque>20</wheelTorque>
 		<!-- Topic to receive geometry_msgs/Twist message commands, defaults to `cmd_vel` -->
 		<commandTopic>cmd_vel</commandTopic>
@@ -329,5 +423,5 @@
 		<odometrySource>1</odometrySource>
 		<!-- Set to true to publish transforms for the wheel links, defaults to false -->
-		<publishWheelTF>false</publishWheelTF>
+		<publishWheelTF>true</publishWheelTF>
 		<!-- Set to true to publish transforms for the odometry, defaults to true -->
 		<publishOdom>true</publishOdom>
@@ -338,40 +432,10 @@
 	  </plugin>
 	</gazebo>
-  <!--========================================== LIDAR PLUGIN - GAZEBO ==========================================-->
-  <!--Sample size of 4000 (original value of RPLidarA1M8) gives an error-->
-  <gazebo reference="laser_link">
-      <!--sensor type="gpu_ray" name="laser"-->
-      <sensor type="ray" name="laser">
-          <pose>0 0 0 0 0 0</pose>
-          <visualize>true</visualize>
-          <update_rate>40</update_rate>
-          <ray>
-              <scan>
-                  <horizontal>
-                      <samples>720</samples>
-                      <resolution>1</resolution>
-                      <min_angle>0</min_angle>
-                      <max_angle>6.28</max_angle>
-                  </horizontal>
-              </scan>
-              <range>
-                  <min>0.1</min>
-                  <max>6</max>
-                  <resolution>0.1</resolution>
-              </range>
-          </ray>
-          <!--plugin name="gpu_laser" filename="libgazebo_ros_gpu_laser.so"-->
-          <plugin name="gpu_laser" filename="libgazebo_ros_laser.so">
-              <topicName>/scan</topicName>
-              <frameName>laser_link</frameName>
-          </plugin>
-      </sensor>
-  </gazebo>
   <!--========================================== JOINT STATE PUBLISHER PLUGIN - GAZEBO ==========================================-->
-     <!--gazebo>
+     <!-- <gazebo>
         <plugin name="joint_state_publisher"
                 filename="libgazebo_ros_joint_state_publisher.so">
-            <jointName>left_wheel_joint, right_wheel_joint, castor_wheel_joint</jointName>
+            <jointName>left_wheel_joint, right_wheel_joint</jointName>
         </plugin>
-    </gazebo-->
+    </gazebo> -->
 </robot>
